Commit message: feat: added slam nodes and modality to work with shelfino1 fixed: TF tree

File: dist_project/models/shelfino_test.xacro (robot description, xacro)
@@ -5,4 +5,11 @@
   <!-- Define the macro for the whole shelfino -->
   <xacro:macro name="shelfino" params='robot_name'>
+    <xacro:if value="${robot_name != 'X'}">
+        <xacro:property name="robot_name_slash" value="'${robot_name}/'" />
+    </xacro:if>
+    <xacro:unless value="${robot_name == 'X'}">
+        <xacro:property name="robot_name_slash" value="''" />
+    </xacro:unless>
+    <xacro:property name="robot_name_slash" value="${robot_name != 'X'}? '' : 'pollo'" />
       <xacro:include filename='shelfino_test/materials.xacro' />
       <xacro:include filename='shelfino_test/shelfino_body.xacro' />

File: dist_project/models/shelfino_test/lidar.xacro (robot description, xacro)
@@ -40,5 +40,5 @@
       <pose> 0 0 0 0 0 0 </pose>
       <visualize>false</visualize>
-      <update_rate>10</update_rate>
+      <update_rate>4</update_rate>
       <ray>
         <scan>

File: dist_project/models/shelfino_test/shelfino_body.xacro (robot description, xacro)
@@ -10,19 +10,19 @@
                   SHELFINO'S BODY
   -->
-  <xacro:property name='body_width' value='0.5'/>
-  <xacro:property name='body_length' value='0.5'/>
-  <xacro:property name='body_height' value='0.4'/>
-  <xacro:property name='body_offset_x' value='0'/>
-  <xacro:property name='body_offset_y' value='0'/>
-  <xacro:property name='body_offset_z' value='0.3'/>
-  <xacro:property name='caster_radius' value='0.05'/>
-  <xacro:property name='caster_width' value='0.05'/>
-  <xacro:property name='caster_offset_z' value='0.1'/>
-  <xacro:property name='body_weight' value='0.5'/>
+  <xacro:property name='body_width' value='0.5' />
+  <xacro:property name='body_length' value='0.5' />
+  <xacro:property name='body_height' value='0.4' />
+  <xacro:property name='body_offset_x' value='0' />
+  <xacro:property name='body_offset_y' value='0' />
+  <xacro:property name='body_offset_z' value='0.3' />
+  <xacro:property name='caster_radius' value='0.05' />
+  <xacro:property name='caster_width' value='0.05' />
+  <xacro:property name='caster_offset_z' value='0.1' />
+  <xacro:property name='body_weight' value='0.5' />
   <link name='${robot_name}/chassis_link'>
     <visual name='body_visual'>
-      <origin xyz='${body_offset_x} ${body_offset_y} ${body_offset_z}'/>
+      <origin xyz='${body_offset_x} ${body_offset_y} ${body_offset_z}' />
       <geometry>
-        <box size='${body_width} ${body_length} ${body_height}'/>
+        <box size='${body_width} ${body_length} ${body_height}' />
       </geometry>
       <xacro:if value="${robot_name == 'evader'}">
@@ -34,28 +34,35 @@
     </visual>
     <visual name='front_caster_visual'>
-      <origin xyz='-0.2 0 ${caster_offset_z}' rpy='0 ${PI_2} ${PI_2}'/>
+      <origin xyz='-0.2 0 ${caster_offset_z}' rpy='0 ${PI_2} ${PI_2}' />
       <geometry>
-        <cylinder radius='${caster_radius}' length='${caster_width}'/>
+        <cylinder radius='${caster_radius}' length='${caster_width}' />
       </geometry>
       <material name='Black' />
     </visual>
     <visual name='back_caster_visual'>
-      <origin xyz='0.2 0 ${caster_offset_z}' rpy='0 ${PI_2} ${PI_2}'/>
+      <origin xyz='0.2 0 ${caster_offset_z}' rpy='0 ${PI_2} ${PI_2}' />
       <geometry>
-        <cylinder radius='${caster_radius}' length='${caster_width}'/>
+        <cylinder radius='${caster_radius}' length='${caster_width}' />
       </geometry>
       <material name='Black' />
     </visual>
     <collision>
-      <origin xyz='${body_offset_x} ${body_offset_y} ${body_offset_z}'/>
+      <origin xyz='${body_offset_x} ${body_offset_y} ${body_offset_z}' />
       <geometry>
-        <box size='${body_width+caster_radius+0.02} ${body_length+0.02} ${body_height+caster_radius*2.0}' />
+        <box
+                    size='${body_width+caster_radius+0.02} ${body_length+0.02} ${body_height+caster_radius*2.0}'
+                />
       </geometry>
     </collision>
     <inertial>
-      <mass value='${body_weight}'/>
-      <inertia ixx='0.001' ixy='0.0' ixz='0.0'
-                iyy='0.001' iyz='0.0'
-                izz='0.001' />
+      <mass value='${body_weight}' />
+      <inertia
+                ixx='0.001'
+                ixy='0.0'
+                ixz='0.0'
+                iyy='0.001'
+                iyz='0.0'
+                izz='0.001'
+            />
     </inertial>
   </link>
@@ -64,12 +71,12 @@
   -->
   <joint name='${robot_name}/base_to_chassis_joint' type='fixed'>
-    <parent link='${robot_name}/base_link'/>
-    <child link='${robot_name}/chassis_link'/>
-    <origin xyz='0 0 0' rpy='0 0 0'/>
+    <parent link='${robot_name}/base_link' />
+    <child link='${robot_name}/chassis_link' />
+    <origin xyz='0 0 0' rpy='0 0 0' />
   </joint>
   <joint name='${robot_name}/base_to_base_footprint_joint' type='fixed'>
-    <parent link='${robot_name}/base_link'/>
-    <child link='${robot_name}/base_footprint'/>
-    <origin xyz='0 0 0' rpy='0 0 0'/>
+    <parent link='${robot_name}/base_link' />
+    <child link='${robot_name}/base_footprint' />
+    <origin xyz='0 0 0' rpy='0 0 0' />
   </joint>
   <!--
@@ -83,6 +90,6 @@
       <material>Gazebo/Green</material>
     </xacro:if>
-    <mu1 value="0.000001"/>
-    <mu2 value="0.000001"/>
+    <mu1 value="0.000001" />
+    <mu2 value="0.000001" />
   </gazebo>
 </robot>

File: dist_project/models/shelfino_test/wheels.xacro (robot description, xacro)
@@ -1,6 +1,6 @@
 <?xml version='1.0' ?>
 <robot name='shelfino' xmlns:xacro='http://www.ros.org/wiki/xacro'>
-  <xacro:property name='wheel_radius' value='0.125'/>
-  <xacro:property name='wheel_width' value='0.03'/>
+  <xacro:property name='wheel_radius' value='0.125' />
+  <xacro:property name='wheel_width' value='0.03' />
   <xacro:macro name="wheel" params="prefix reflect">
     <!--
@@ -10,18 +10,23 @@
       <visual>
         <geometry>
-          <cylinder radius="${wheel_radius}" length="${wheel_width}"/>
+          <cylinder radius="${wheel_radius}" length="${wheel_width}" />
         </geometry>
-        <material name="Black"/>
+        <material name="Black" />
       </visual>
       <collision>
         <geometry>
-          <cylinder radius="${wheel_radius}" length="${wheel_width+0.005}"/>
+          <cylinder radius="${wheel_radius}" length="${wheel_width+0.005}" />
         </geometry>
       </collision>
       <inertial>
-        <mass value="0.028498940"/>
-        <inertia ixx='1.1175580e-05' ixy='-4.2369783e-11' ixz='-5.9381719e-09'
-            iyy='1.1192413e-05' iyz='-1.4400107e-11'
-            izz='2.0712558e-05' />
+        <mass value="0.028498940" />
+        <inertia
+                    ixx='1.1175580e-05'
+                    ixy='-4.2369783e-11'
+                    ixz='-5.9381719e-09'
+                    iyy='1.1192413e-05'
+                    iyz='-1.4400107e-11'
+                    izz='2.0712558e-05'
+                />
       </inertial>
     </link>
@@ -30,8 +35,13 @@
     -->
     <joint name="${robot_name}/${prefix}_wheel_joint" type="continuous">
-      <parent link="${robot_name}/chassis_link"/>
-      <child link="${robot_name}/${prefix}_wheel"/>
-      <origin xyz="0 ${reflect*(body_width/2+0.02)} ${wheel_radius+0.05}" rpy="0 ${pi/2} ${pi/2}"/>
-      <axis xyz="0 0 1"/> <!-- specifies the axis around which it should revolve -->
+      <parent link="${robot_name}/chassis_link" />
+      <child link="${robot_name}/${prefix}_wheel" />
+      <origin
+                xyz="0 ${reflect*(body_width/2+0.02)} ${wheel_radius+0.05}"
+                rpy="0 ${pi/2} ${pi/2}"
+            />
+      <axis
+                xyz="0 0 1"
+            /> <!-- specifies the axis around which it should revolve -->
     </joint>
     <!--
@@ -40,5 +50,8 @@
     <gazebo reference="${robot_name}/${prefix}_wheel">
       <material>Gazebo/Black</material>
-      <plugin name='gazebo_ros_joint_state_publisher' filename='libgazebo_ros_joint_state_publisher.so'>
+      <plugin
+                name='gazebo_ros_joint_state_publisher'
+                filename='libgazebo_ros_joint_state_publisher.so'
+            >
         <update_rate>100</update_rate>
         <ros>

File: dist_project/models/shelfino_test/xmas_hat.xacro (robot description, xacro)
@@ -5,10 +5,13 @@
     <visual name='visual'>
       <geometry>
-        <mesh filename='package://shelfino_description/models/xmas_hat/meshes/xmas_hat.dae' scale='0.01 0.01 0.01'/>
+        <mesh
+                    filename='package://shelfino_description/models/xmas_hat/meshes/xmas_hat.dae'
+                    scale='0.01 0.01 0.01'
+                />
       </geometry>
     </visual>
     <collision name='collision'>
       <geometry>
-        <cylinder radius='0.01' length='0.01'/>
+        <cylinder radius='0.01' length='0.01' />
         <!-- <mesh filename='package://shelfino_description/models/xmas_hat/meshes/xmas_hat.dae' scale='0.01 0.01 0.01'/> -->
       </geometry>
@@ -16,7 +19,7 @@
   </link>
   <joint name='${robot_name}/hat_joint' type='fixed'>
-    <parent link='${robot_name}/base_link'/>
-    <child link='${robot_name}/hat'/>
-    <origin xyz='0 0 ${body_height+0.1}' rpy='0 0 0'/>
+    <parent link='${robot_name}/base_link' />
+    <child link='${robot_name}/hat' />
+    <origin xyz='0 0 ${body_height+0.1}' rpy='0 0 0' />
   </joint>
 </robot>

Commit message: feat: added cluster filtering

File: dist_project/models/shelfino_test.xacro (robot description, xacro)
@@ -2,14 +2,8 @@
 <robot name='shelfino' xmlns:xacro='http://www.ros.org/wiki/xacro'>
   <xacro:property name='PI_2' value='1.5707963267948966' />
+  <xacro:arg name="max_camera_depth" default="8.0" />
   <xacro:arg name="robot_name" default="X" />
   <!-- Define the macro for the whole shelfino -->
-  <xacro:macro name="shelfino" params='robot_name'>
-    <xacro:if value="${robot_name != 'X'}">
-        <xacro:property name="robot_name_slash" value="'${robot_name}/'" />
-    </xacro:if>
-    <xacro:unless value="${robot_name == 'X'}">
-        <xacro:property name="robot_name_slash" value="''" />
-    </xacro:unless>
-    <xacro:property name="robot_name_slash" value="${robot_name != 'X'}? '' : 'pollo'" />
+  <xacro:macro name="shelfino" params='robot_name max_camera_depth'>
       <xacro:include filename='shelfino_test/materials.xacro' />
       <xacro:include filename='shelfino_test/shelfino_body.xacro' />
@@ -22,4 +16,4 @@
   </xacro:macro>
   <!-- Instantiate the model -->
-  <xacro:shelfino robot_name="$(arg robot_name)" />
+  <xacro:shelfino robot_name="$(arg robot_name)" max_camera_depth="$(arg max_camera_depth)" />
 </robot>

File: dist_project/models/shelfino_test/frontal_camera.xacro (robot description, xacro)
@@ -53,5 +53,5 @@
         <horizontal_fov>1.089</horizontal_fov>
         <image>
-            <format>R8G8B8</format>
+            <format>B8G8R8</format>
             <width>640</width>
             <heigth>480</heigth>
@@ -59,5 +59,5 @@
         <clip>
             <near>0.05</near>
-            <far>8.00</far>
+            <far>${max_camera_depth}</far>
         </clip>
       </camera>
