Commit message: generato i grafici per i dati raccolti di coordination, ruotata la camera dello shelfino e spsostata un pò più in su fixxato un commit in bring up shelfino

File: dist_project/models/shelfino_test/frontal_camera.xacro (robot description, xacro)
@@ -36,5 +36,5 @@
     <parent link='${robot_name}/chassis_link' />
     <child link='${robot_name}/frontal_camera_link' />
-    <origin xyz='${body_length/2+0.10} 0 ${body_height/2}' rpy='0 0 0' />
+    <origin xyz='${body_length/2+0.10} 0 ${body_height/2+0.7}' rpy='0 0.087 0' />
   </joint>
   <!-- From Ros Joint system to video coordinate system -->
